Commit message: Rear and Front wheels controlls working mecanum drive controller testing is pending

File: src/mecanum_robot_hardware/description/urdf/AruBot.urdf (robot description, URDF)
Before this commit: robot AruBot, 5 links, 4 joints
Links:
- link front_left_wheel: geometry visual cylinder length=0.029 radius=0.0325
- link front_right_wheel: geometry visual cylinder length=0.029 radius=0.0325
- link rear_left_wheel: geometry visual cylinder length=0.029 radius=0.0325
- link rear_right_wheel: geometry visual cylinder length=0.029 radius=0.0325
Joints:
- joint base_link_front_right_wheel: origin xyz=0.07145 -0.136701 -0.051657 rpy=1.57 0 0 -> xyz=0.07145 -0.136701 -0.051657 rpy=-1.57 0 0
- joint base_link_rear_right_wheel: origin xyz=-0.08355 -0.136701 -0.051657 rpy=1.57 0 0 -> xyz=-0.08355 -0.136701 -0.051657 rpy=-1.57 0 0

File: src/ros2_control_demo_description/diffbot/urdf/diffbot_description.urdf.xacro (robot description, xacro)
@@ -10,5 +10,5 @@
   <xacro:property name="wheel_mass" value="0.3" /> <!-- arbitrary value for wheel mass -->
   <xacro:property name="wheel_len" value="0.029" />
-  <xacro:property name="wheel_radius" value="0.065" />
+  <xacro:property name="wheel_radius" value="0.0325" />
   <xacro:property name="caster_wheel_mass" value="0.1" /> <!-- arbitrary value for caster wheel mass -->
   <xacro:property name="caster_wheel_radius" value="0.015" />
@@ -105,5 +105,5 @@
     <parent link="${prefix}base_link"/>
     <child link="${prefix}rear_right_wheel"/>
-    <origin xyz="-0.08355 -0.136701 -0.051657" rpy="${PI/2} 0 0"/>
+    <origin xyz="-0.08355 -0.136701 -0.051657" rpy="${-PI/2} 0 0"/>
     <axis xyz="0 0 1"/>
     <limit effort="100" velocity="1.0"/>
@@ -117,9 +117,9 @@
     <limit effort="100" velocity="1.0"/>
   </joint>
-  <!-- front left wheel joint-->
+  <!-- front right wheel joint-->
   <joint name="${prefix}front_right_wheel_joint" type="continuous">
     <parent link="${prefix}base_link"/>
     <child link="${prefix}front_right_wheel"/>
-    <origin xyz="0.07145 -0.136701 -0.051657" rpy="${PI/2} 0 0"/>
+    <origin xyz="0.07145 -0.136701 -0.051657" rpy="${-PI/2} 0 0"/>
     <axis xyz="0 0 1"/>
     <limit effort="100" velocity="1.0"/>
