Commit message: Working hardware controller and a launch file along with slam toolbox parameter file

File: src/ros2_control_demo_description/diffbot/urdf/diffbot_description.urdf.xacro (robot description, xacro)
@@ -93,4 +93,19 @@
     </visual>
   </link>
+  <!-- Lidar Link-->
+  <link name="${prefix}laser">
+    <collision>
+      <origin xyz="0 0 0" rpy= "0 0 0"/>
+      <geometry>
+        <cylinder length="0.02" radius="0.07"/>
+      </geometry>
+    </collision>
+    <visual>
+      <origin xyz="0 0 0" rpy= "0 0 0"/>
+      <geometry>
+        <cylinder length="0.02" radius="0.07"/>
+      </geometry>
+    </visual>
+  </link>
   <!-- rear left wheel joint-->
   <joint name="${prefix}rear_left_wheel_joint" type="continuous">
@@ -125,4 +140,10 @@
     <limit effort="100" velocity="1.0"/>
   </joint>
+  <!-- Lidar joint-->
+  <joint name="${prefix}lidar_link_joint" type="fixed">
+    <parent link="${prefix}base_link"/>
+    <child link="${prefix}laser"/>
+    <origin xyz = "0.02435 0 0.176" rpy = "0 0 0"/>
+  </joint>
   </xacro:macro>
 </robot>

Commit message: Integration till close to package

File: src/ros2_control_demo_description/diffbot/urdf/diffbot_description.urdf.xacro (robot description, xacro)
@@ -5,5 +5,5 @@
   <xacro:property name="PI" value="3.1415926535897931"/>
   <xacro:property name="base_mass" value="0.3" /> <!-- arbitrary value for base mass -->
-  <xacro:property name="base_width" value="0.2513" />
+  <xacro:property name="base_width" value="0.2713" />
   <xacro:property name="base_length" value="0.2" />
   <xacro:property name="base_height" value="0.005" />
@@ -112,5 +112,5 @@
     <parent link="${prefix}base_link"/>
     <child link="${prefix}rear_left_wheel"/>
-    <origin xyz="-0.08355 0.136701 -0.051657" rpy="${-PI/2} 0 0"/>
+    <origin xyz="-0.09355 0.136701 -0.051657" rpy="${-PI/2} 0 0"/>
     <axis xyz="0 0 1"/>
     <limit effort="100" velocity="1.0"/>
@@ -120,5 +120,5 @@
     <parent link="${prefix}base_link"/>
     <child link="${prefix}rear_right_wheel"/>
-    <origin xyz="-0.08355 -0.136701 -0.051657" rpy="${-PI/2} 0 0"/>
+    <origin xyz="-0.09355 -0.136701 -0.051657" rpy="${PI/2} 0 0"/>
     <axis xyz="0 0 1"/>
     <limit effort="100" velocity="1.0"/>
@@ -128,5 +128,5 @@
     <parent link="${prefix}base_link"/>
     <child link="${prefix}front_left_wheel"/>
-    <origin xyz="0.07145 0.136701 -0.051657" rpy="${-PI/2} 0 0"/>
+    <origin xyz="0.08145 0.136701 -0.051657" rpy="${-PI/2} 0 0"/>
     <axis xyz="0 0 1"/>
     <limit effort="100" velocity="1.0"/>
@@ -136,5 +136,5 @@
     <parent link="${prefix}base_link"/>
     <child link="${prefix}front_right_wheel"/>
-    <origin xyz="0.07145 -0.136701 -0.051657" rpy="${-PI/2} 0 0"/>
+    <origin xyz="0.08145 -0.136701 -0.051657" rpy="${PI/2} 0 0"/>
     <axis xyz="0 0 1"/>
     <limit effort="100" velocity="1.0"/>
@@ -144,5 +144,5 @@
     <parent link="${prefix}base_link"/>
     <child link="${prefix}laser"/>
-    <origin xyz = "0.02435 0 0.176" rpy = "0 0 0"/>
+    <origin xyz = "0.01435 0 0.176" rpy = "0 0 0"/>
   </joint>
   </xacro:macro>
